File: HandCHime.kicad_sch (KiCad schematic)
At the start: 18 parts, among them J1 USB_C_Receptacle_USB2.0, J2 Pins, SW0 BOOT, SW1 Row 0, Col 0, SW2 Row 0, Col 1, U1 CH552T, U2 USBLC6-2P6

Commit message: Fix part numbers for recently updated components
Parts:
- R3: DigiKey 311-10.0KHR -> 311-5.10KHR; LCSC C25804 -> C23186
- SW0: DigiKey 4809-SKQGABE010 -> SW1020CT-ND; LCSC C115351 -> C231329
Changed lines of the file:
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@@
 			)
 		)
-		(property "LCSC" "C25804"
+		(property "LCSC" "C23186"
 			(at 223.52 81.28 90)
 			(effects
@@
 			)
 		)
-		(property "DigiKey" "311-10.0KHR"
+		(property "DigiKey" "311-5.10KHR"
 			(at 223.52 81.28 90)
 			(effects
@@
 			)
 		)
-		(property "LCSC" "C115351"
+		(property "LCSC" "C231329"
 			(at 234.95 81.28 0)
 			(effects
@@
 			)
 		)
-		(property "DigiKey" "4809-SKQGABE010"
+		(property "DigiKey" "SW1020CT-ND"
 			(at 234.95 81.28 0)
 			(effects
