File: Handchime.kicad_sch (KiCad schematic)
At the start: 24 parts, among them J1 USB_C_Receptacle_USB2.0_16P, J2 Pins, J3 SWD, SW0 BOOT, SW1 Row 0, Col 0, SW2 Row 0, Col 1, U1 STM32C071GBUx, U2 PRTR5V0U2X, U3 XC6206P332MR-G

Commit message: Change name to HandSTamp
Other:
- company: u/bgkendall -> bgkendall
- title: ISOCHet -> HandSTaMp
Changed lines of the file:
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@@
 	(paper "A4")
 	(title_block
-		(title "ISOCHet")
-		(date "2024-04-24")
-		(rev "v1.0")
-		(company "u/bgkendall")
+		(title "HandSTaMp")
+		(date "2026-04-11")
+		(rev "v2.0")
+		(company "bgkendall")
 	)
 	(text "Keys"
