File: HandSTaMp.kicad_pcb (KiCad board)
At the start: 2 copper layers, 40.6 x 16.5 mm, 24 parts, among them J1 USB_C_Receptacle_USB2.0_16P, J2 Pins, J3 SWD, SW0 BOOT, SW1 Row 0, Col 0, SW2 Row 0, Col 1, U1 STM32C071GBUx, U2 PRTR5V0U2X, U3 XC6206P332MR-G

Commit message: Update filenames and libraries
Parts:
- J2: footprint Project Library:Handchime -> Project Library:HandSTaMp
Changed lines of the file:
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@@
 		(property ki_fp_filters "QFN*4x4mm*P0.5mm*")
 		(sheetname "/")
-		(sheetfile "Handchime.kicad_sch")
+		(sheetfile "HandSTaMp.kicad_sch")
 		(units
 			(unit
@@
 		(property ki_fp_filters "USB*C*Receptacle*")
 		(sheetname "/")
-		(sheetfile "Handchime.kicad_sch")
+		(sheetfile "HandSTaMp.kicad_sch")
 		(units
 			(unit
@@
 		(property ki_fp_filters "C_*")
 		(sheetname "/")
-		(sheetfile "Handchime.kicad_sch")
+		(sheetfile "HandSTaMp.kicad_sch")
 		(units
 			(unit
@@
 		(property ki_fp_filters "C_*")
 		(sheetname "/")
-		(sheetfile "Handchime.kicad_sch")
+		(sheetfile "HandSTaMp.kicad_sch")
 		(units
 			(unit
@@
 		(property ki_fp_filters "R_*")
 		(sheetname "/")
-		(sheetfile "Handchime.kicad_sch")
+		(sheetfile "HandSTaMp.kicad_sch")
 		(units
 			(unit
@@
 		(property ki_fp_filters "SOT?143*")
 		(sheetname "/")
-		(sheetfile "Handchime.kicad_sch")
+		(sheetfile "HandSTaMp.kicad_sch")
 		(units
 			(unit
@@
 		(property ki_fp_filters "*polyfuse* *PTC*")
 		(sheetname "/")
-		(sheetfile "Handchime.kicad_sch")
+		(sheetfile "HandSTaMp.kicad_sch")
 		(units
 			(unit
@@
 		)
 		(sheetname "/")
-		(sheetfile "Handchime.kicad_sch")
+		(sheetfile "HandSTaMp.kicad_sch")
 		(units
 			(unit
@@
 		(property ki_fp_filters "TO-???* *_Diode_* *SingleDiode* D_*")
 		(sheetname "/")
-		(sheetfile "Handchime.kicad_sch")
+		(sheetfile "HandSTaMp.kicad_sch")
 		(units
 			(unit
@@
 		(property ki_fp_filters "SOT?23?3*")
 		(sheetname "/")
-		(sheetfile "Handchime.kicad_sch")
+		(sheetfile "HandSTaMp.kicad_sch")
 		(units
 			(unit
@@
 		(property ki_fp_filters "C_*")
 		(sheetname "/")
-		(sheetfile "Handchime.kicad_sch")
+		(sheetfile "HandSTaMp.kicad_sch")
 		(units
 			(unit
@@
 		(property ki_fp_filters "TO-???* *_Diode_* *SingleDiode* D_*")
 		(sheetname "/")
-		(sheetfile "Handchime.kicad_sch")
+		(sheetfile "HandSTaMp.kicad_sch")
 		(units
 			(unit
@@
 		(property ki_fp_filters "R_*")
 		(sheetname "/")
-		(sheetfile "Handchime.kicad_sch")
+		(sheetfile "HandSTaMp.kicad_sch")
 		(units
 			(unit
@@
 		(property ki_fp_filters "C_*")
 		(sheetname "/")
-		(sheetfile "Handchime.kicad_sch")
+		(sheetfile "HandSTaMp.kicad_sch")
 		(units
 			(unit
@@
 		(property ki_fp_filters "Connector*:*_1x??_*")
 		(sheetname "/")
-		(sheetfile "Handchime.kicad_sch")
+		(sheetfile "HandSTaMp.kicad_sch")
 		(units
 			(unit
@@
 		)
 	)
-	(footprint "Project Library:Handchime"
+	(footprint "Project Library:HandSTaMp"
 		(locked yes)
 		(layer "F.Cu")
@@
 		)
 		(sheetname "/")
-		(sheetfile "Handchime.kicad_sch")
+		(sheetfile "HandSTaMp.kicad_sch")
 		(units
 			(unit
@@
 		(property ki_fp_filters "R_*")
 		(sheetname "/")
-		(sheetfile "Handchime.kicad_sch")
+		(sheetfile "HandSTaMp.kicad_sch")
 		(units
 			(unit
@@
 		(property ki_fp_filters "R_*")
 		(sheetname "/")
-		(sheetfile "Handchime.kicad_sch")
+		(sheetfile "HandSTaMp.kicad_sch")
 		(units
 			(unit
@@
 		(property ki_fp_filters "R_*")
 		(sheetname "/")
-		(sheetfile "Handchime.kicad_sch")
+		(sheetfile "HandSTaMp.kicad_sch")
 		(units
 			(unit
@@
 		(property ki_fp_filters "C_*")
 		(sheetname "/")
-		(sheetfile "Handchime.kicad_sch")
+		(sheetfile "HandSTaMp.kicad_sch")
 		(units
 			(unit
@@
 		(property ki_fp_filters "TO-???* *_Diode_* *SingleDiode* D_*")
 		(sheetname "/")
-		(sheetfile "Handchime.kicad_sch")
+		(sheetfile "HandSTaMp.kicad_sch")
 		(units
 			(unit
@@
 		)
 		(sheetname "/")
-		(sheetfile "Handchime.kicad_sch")
+		(sheetfile "HandSTaMp.kicad_sch")
 		(units
 			(unit
@@
 		(property ki_fp_filters "Jumper* TestPoint*2Pads* TestPoint*Bridge*")
 		(sheetname "/")
-		(sheetfile "Handchime.kicad_sch")
+		(sheetfile "HandSTaMp.kicad_sch")
 		(units
 			(unit
@@
 		)
 		(sheetname "/")
-		(sheetfile "Handchime.kicad_sch")
+		(sheetfile "HandSTaMp.kicad_sch")
 		(units
 			(unit
