File: HandSTaMp.kicad_sch (KiCad schematic)
At the start: 24 parts, among them J1 USB_C_Receptacle_USB2.0_16P, J2 Pins, J3 SWD, SW0 BOOT, SW1 Row 0, Col 0, SW2 Row 0, Col 1, U1 STM32C071GBUx, U2 PRTR5V0U2X, U3 XC6206P332MR-G

Commit message: Update filenames and libraries
Parts:
- J2: footprint Project Library:Handchime -> Project Library:HandSTaMp; symbol Project Library:Handchime -> Project Library:HandSTaMp
Changed lines of the file:
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@@
 		)
 		(instances
-			(project "Handchime"
+			(project "HandSTaMp"
 				(path "/34400e51-cf83-464a-b3ec-e9a28a972a27"
 					(reference "D3")
@@
 		)
 		(instances
-			(project "Handchime"
+			(project "HandSTaMp"
 				(path "/34400e51-cf83-464a-b3ec-e9a28a972a27"
 					(reference "#PWR04")
@@
 		)
 		(instances
-			(project "Handchime"
+			(project "HandSTaMp"
 				(path "/34400e51-cf83-464a-b3ec-e9a28a972a27"
 					(reference "C4")
@@
 		)
 		(instances
-			(project "Handchime"
+			(project "HandSTaMp"
 				(path "/34400e51-cf83-464a-b3ec-e9a28a972a27"
 					(reference "U3")
@@
 		)
 		(instances
-			(project "Handchime"
+			(project "HandSTaMp"
 				(path "/34400e51-cf83-464a-b3ec-e9a28a972a27"
 					(reference "SW2")
@@
 		)
 		(instances
-			(project "Handchime"
+			(project "HandSTaMp"
 				(path "/34400e51-cf83-464a-b3ec-e9a28a972a27"
 					(reference "#PWR013")
@@
 		)
 		(instances
-			(project "Handchime"
+			(project "HandSTaMp"
 				(path "/34400e51-cf83-464a-b3ec-e9a28a972a27"
 					(reference "R1")
@@
 		)
 		(instances
-			(project "Handchime"
+			(project "HandSTaMp"
 				(path "/34400e51-cf83-464a-b3ec-e9a28a972a27"
 					(reference "#PWR09")
@@
 		)
 		(instances
-			(project "Handchime"
+			(project "HandSTaMp"
 				(path "/34400e51-cf83-464a-b3ec-e9a28a972a27"
 					(reference "#PWR028")
@@
 		)
 		(instances
-			(project "Handchime"
+			(project "HandSTaMp"
 				(path "/34400e51-cf83-464a-b3ec-e9a28a972a27"
 					(reference "R4")
@@
 		)
 		(instances
-			(project "Handchime"
+			(project "HandSTaMp"
 				(path "/34400e51-cf83-464a-b3ec-e9a28a972a27"
 					(reference "#PWR027")
@@
 		)
 		(instances
-			(project "Handchime"
+			(project "HandSTaMp"
 				(path "/34400e51-cf83-464a-b3ec-e9a28a972a27"
 					(reference "J3")
@@
 		)
 		(instances
-			(project "Handchime"
+			(project "HandSTaMp"
 				(path "/34400e51-cf83-464a-b3ec-e9a28a972a27"
 					(reference "U2")
@@
 		)
 		(instances
-			(project "Handchime"
+			(project "HandSTaMp"
 				(path "/34400e51-cf83-464a-b3ec-e9a28a972a27"
 					(reference "#PWR07")
@@
 		)
 		(instances
-			(project "Handchime"
+			(project "HandSTaMp"
 				(path "/34400e51-cf83-464a-b3ec-e9a28a972a27"
 					(reference "#PWR01")
@@
 		)
 		(instances
-			(project "Handchime"
+			(project "HandSTaMp"
 				(path "/34400e51-cf83-464a-b3ec-e9a28a972a27"
 					(reference "U1")
@@
 		)
 		(instances
-			(project "Handchime"
+			(project "HandSTaMp"
 				(path "/34400e51-cf83-464a-b3ec-e9a28a972a27"
 					(reference "#PWR0102")
@@
 		)
 		(instances
-			(project "Handchime"
+			(project "HandSTaMp"
 				(path "/34400e51-cf83-464a-b3ec-e9a28a972a27"
 					(reference "#PWR030")
@@
 		)
 		(instances
-			(project "Handchime"
+			(project "HandSTaMp"
 				(path "/34400e51-cf83-464a-b3ec-e9a28a972a27"
 					(reference "#PWR019")
@@
 		)
 		(instances
-			(project "Handchime"
+			(project "HandSTaMp"
 				(path "/34400e51-cf83-464a-b3ec-e9a28a972a27"
 					(reference "#PWR031")
@@
 		)
 		(instances
-			(project "Handchime"
+			(project "HandSTaMp"
 				(path "/34400e51-cf83-464a-b3ec-e9a28a972a27"
 					(reference "#PWR08")
@@
 		)
 		(instances
-			(project "Handchime"
+			(project "HandSTaMp"
 				(path "/34400e51-cf83-464a-b3ec-e9a28a972a27"
 					(reference "SW0")
@@
 		)
 		(instances
-			(project "Handchime"
+			(project "HandSTaMp"
 				(path "/34400e51-cf83-464a-b3ec-e9a28a972a27"
 					(reference "D1")
@@
 		)
 		(instances
-			(project "Handchime"
+			(project "HandSTaMp"
 				(path "/34400e51-cf83-464a-b3ec-e9a28a972a27"
 					(reference "F1")
@@
 		)
 		(instances
-			(project "Handchime"
+			(project "HandSTaMp"
 				(path "/34400e51-cf83-464a-b3ec-e9a28a972a27"
 					(reference "#PWR029")
@@
 		)
 		(instances
-			(project "Handchime"
+			(project "HandSTaMp"
 				(path "/34400e51-cf83-464a-b3ec-e9a28a972a27"
 					(reference "D2")
@@
 		)
 		(instances
-			(project "Handchime"
+			(project "HandSTaMp"
 				(path "/34400e51-cf83-464a-b3ec-e9a28a972a27"
 					(reference "C5")
@@
 		)
 		(instances
-			(project "Handchime"
+			(project "HandSTaMp"
 				(path "/34400e51-cf83-464a-b3ec-e9a28a972a27"
 					(reference "C1")
@@
 		)
 		(instances
-			(project "Handchime"
+			(project "HandSTaMp"
 				(path "/34400e51-cf83-464a-b3ec-e9a28a972a27"
 					(reference "#PWR011")
@@
 		)
 		(instances
-			(project "Handchime"
+			(project "HandSTaMp"
 				(path "/34400e51-cf83-464a-b3ec-e9a28a972a27"
 					(reference "#PWR012")
@@
 		)
 		(instances
-			(project "Handchime"
+			(project "HandSTaMp"
 				(path "/34400e51-cf83-464a-b3ec-e9a28a972a27"
 					(reference "R3")
@@
 		)
 		(instances
-			(project "Handchime"
+			(project "HandSTaMp"
 				(path "/34400e51-cf83-464a-b3ec-e9a28a972a27"
 					(reference "SW1")
@@
 		)
 		(instances
-			(project "Handchime"
+			(project "HandSTaMp"
 				(path "/34400e51-cf83-464a-b3ec-e9a28a972a27"
 					(reference "#PWR025")
@@
 		)
 		(instances
-			(project "Handchime"
+			(project "HandSTaMp"
 				(path "/34400e51-cf83-464a-b3ec-e9a28a972a27"
 					(reference "C2")
@@
 		)
 		(instances
-			(project "Handchime"
+			(project "HandSTaMp"
 				(path "/34400e51-cf83-464a-b3ec-e9a28a972a27"
 					(reference "R5")
@@
 		)
 		(instances
-			(project "Handchime"
+			(project "HandSTaMp"
 				(path "/34400e51-cf83-464a-b3ec-e9a28a972a27"
 					(reference "#PWR024")
@@
 		)
 		(instances
-			(project "Handchime"
+			(project "HandSTaMp"
 				(path "/34400e51-cf83-464a-b3ec-e9a28a972a27"
 					(reference "#PWR026")
@@
 		)
 		(instances
-			(project "Handchime"
+			(project "HandSTaMp"
 				(path "/34400e51-cf83-464a-b3ec-e9a28a972a27"
 					(reference "#PWR03")
@@
 		)
 		(instances
-			(project "Handchime"
+			(project "HandSTaMp"
 				(path "/34400e51-cf83-464a-b3ec-e9a28a972a27"
 					(reference "#PWR010")
@@
 		)
 		(instances
-			(project "Handchime"
+			(project "HandSTaMp"
 				(path "/34400e51-cf83-464a-b3ec-e9a28a972a27"
 					(reference "#PWR02")
@@
 		)
 		(instances
-			(project "Handchime"
+			(project "HandSTaMp"
 				(path "/34400e51-cf83-464a-b3ec-e9a28a972a27"
 					(reference "#PWR022")
@@
 		)
 		(instances
-			(project "Handchime"
+			(project "HandSTaMp"
 				(path "/34400e51-cf83-464a-b3ec-e9a28a972a27"
 					(reference "#PWR014")
@@
 		)
 		(instances
-			(project "Handchime"
+			(project "HandSTaMp"
 				(path "/34400e51-cf83-464a-b3ec-e9a28a972a27"
 					(reference "#PWR032")
@@
 	)
 	(symbol
-		(lib_id "Project Library:Handchime")
+		(lib_id "Project Library:HandSTaMp")
 		(at 204.47 139.7 0)
 		(unit 1)
@@
 			)
 		)
-		(property "Footprint" "Project Library:Handchime"
+		(property "Footprint" "Project Library:HandSTaMp"
 			(at 204.47 139.7 0)
 			(hide yes)
@@
 		)
 		(instances
-			(project "Handchime"
+			(project "HandSTaMp"
 				(path "/34400e51-cf83-464a-b3ec-e9a28a972a27"
 					(reference "J2")
@@
 		)
 		(instances
-			(project "Handchime"
+			(project "HandSTaMp"
 				(path "/34400e51-cf83-464a-b3ec-e9a28a972a27"
 					(reference "NT1")
@@
 		)
 		(instances
-			(project "Handchime"
+			(project "HandSTaMp"
 				(path "/34400e51-cf83-464a-b3ec-e9a28a972a27"
 					(reference "R2")
@@
 		)
 		(instances
-			(project "Handchime"
+			(project "HandSTaMp"
 				(path "/34400e51-cf83-464a-b3ec-e9a28a972a27"
 					(reference "C3")
@@
 		)
 		(instances
-			(project "Handchime"
+			(project "HandSTaMp"
 				(path "/34400e51-cf83-464a-b3ec-e9a28a972a27"
 					(reference "J1")
